File: ACB/ACB/ACB-R1.0-43-CH09/ACB-R1.1.sch (EAGLE design)
At the start: 430 parts, among them IC1 PIC32MX470F512L-I/PF, IC10 MAX9938HEUK+T, IC11 24LC32A-I/MS, IC12 SN65HVD12D, IC13 REF3025, IC14 TPD2E001DZDR, IC15 TPD2E001DZDR, IC16 MCP6042-I/MS, IC17 L6227Q, IC18 DS2431, IC2 R1LV1616, IC201 DS2431, IC3 74LVC573APW-TSSOP20, IC4 74LVC573APW-TSSOP20, IC5 TLV73315PDBV, IC6 MIC841LYC, IC7 24LC32A-I/MS, IC8 LT3971EMSE, IC9 AT25SF321-SSHD, J1 FH12A-24S-0.5SH, J10 3-641215-2, J11 DNP-DM3AT, J12 USB_A_180, J14 pin1x8, J15 pin2x8, J17 DNP-open-hole, J2 FH12A-24S-0.5SH, J3 RJ8-8-180, J4 RJ8-8-180, J5 MOLEX430450613, J6 MOLEX430450613, J7 3-641215-2, J8 3-641215-2, J9 3-641215-2, Q1 SSM6P49NU,LFPZ, Q10 FDG6303N, Q11 FDG6303N, Q12 FDG6303N, Q13 FDG6303N, Q14 FDG6303N, Q2 SSM6P49NU,LFPZ, Q3 FDG6303N, Q4 FDG6303N, Q5 FDC6506P, Q6 FDC6506P, Q7 FDG6303N, Q8 FDC6506P, Q9 FDG6303N, T1 PIC-OUT, T10 PIC-RPX, T11 PIC-RPX, T12 PIC-RPX, T13 PIC-RPX, T14 PIC-RPX, T15 PIC-OUT, T16 PIC-RPX, T17 PIC-RPX, T18 PIC-RPX, T19 PIC-RPX, T2 PIC-OUT, T20 PIC-OUT, T21 PIC-OUT, T22 PIC-RPX, T23 PIC-RPX, T24 PIC-RPX, T25 PIC-OUT, T26 PIC-OUT, T27 PIC-OUT, T28 PIC-OUT, T29 PIC-OUT, T3 PIC-RPX, T30 PIC-OUT, T31 PIC-OUT, T32 PIC-OUT, T33 PIC-OUT, T34 PIC-RPX, T35 PIC-RPX, T36 PIC-OUT, T37 PIN-AN, T38 PIN-AN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

Commit message: quick edit
renamed some nets for the ACB
Connections:
- net D+ renamed D_P
- net D- renamed D_N
Other:
- note added: "find connector for door sensor"
- note added: "find connector for motor"
- moved on the sheet: C201, C89, C90, C91, C92-1, C93, C94, C95, D1, D10, D201, D8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

Commit message: addedd some info to the SCH
Other:
- note added: "G5 MOTOR DRIVER CIRCUIT"
- note added: "GEAR MOTOR BOARD"
Changed lines of the file:
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@@
 <text x="-76.2" y="265.176" size="0.889" layer="95">prechodovy pri ADON,REFEN=0-&gt;1 cca 250us</text>
 <text x="-76.2" y="263.906" size="0.889" layer="95">tzn. pri odberu cca 0,22mA</text>
-<text x="-142.24" y="332.74" size="1.778" layer="95">V datshitu DS60001185F-page 318 je uvedeno,
+<text x="-152.4" y="332.74" size="1.778" layer="95">V datshitu DS60001185F-page 318 je uvedeno,
 ze AN15-AN27 jsou na hovno....  pice...
 CURR-SENSE je na AN19
@@
 <text x="706.12" y="670.56" size="1.778" layer="97">find connector for door sensor</text>
 <text x="698.5" y="579.12" size="1.778" layer="97">find connector for door sensor</text>
+<wire x1="619.76" y1="683.26" x2="619.76" y2="495.3" width="0.1524" layer="94" style="shortdash"/>
+<wire x1="619.76" y1="495.3" x2="767.08" y2="495.3" width="0.1524" layer="94" style="shortdash"/>
+<wire x1="767.08" y1="495.3" x2="767.08" y2="683.26" width="0.1524" layer="94" style="shortdash"/>
+<wire x1="767.08" y1="683.26" x2="619.76" y2="683.26" width="0.1524" layer="94" style="shortdash"/>
+<wire x1="619.76" y1="495.3" x2="350.52" y2="495.3" width="0.1524" layer="94" style="shortdash"/>
+<wire x1="350.52" y1="495.3" x2="350.52" y2="683.26" width="0.1524" layer="94" style="shortdash"/>
+<wire x1="350.52" y1="683.26" x2="619.76" y2="683.26" width="0.1524" layer="94" style="shortdash"/>
+<text x="764.54" y="505.46" size="6.4516" layer="94" rot="R180">GEAR MOTOR BOARD</text>
+<text x="617.22" y="505.46" size="6.4516" layer="94" rot="R180">G5 MOTOR DRIVER CIRCUIT</text>
 </plain>
 <instances>
