File: ACB/ACB/ACB-R1.0-43-CH09/ACB Jr..sch (EAGLE design)
At the start: 384 parts, among them IC1 PIC32MX470F512L-I/PF, IC10 MAX9938HEUK+T, IC11 24LC32A-I/MS, IC12 SN65HVD12D, IC13 REF3025, IC14 TPD2E001DZDR, IC15 TPD2E001DZDR, IC16 MCP6042-I/MS, IC2 R1LV1616, IC3 74LVC573APW-TSSOP20, IC4 74LVC573APW-TSSOP20, IC5 TLV73315PDBV, IC6 MIC841LYC, IC7 24LC32A-I/MS, IC8 LT3971EMSE, IC9 AT25SF321-SSHD, J1 FH12A-24S-0.5SH, J10 3-641215-2, J11 DNP-DM3AT, J12 USB_A_180, J14 pin1x8, J15 pin2x8, J17 DNP-open-hole, J2 FH12A-24S-0.5SH, J3 RJ8-8-180, J4 RJ8-8-180, J5 MOLEX430450613, J6 MOLEX430450613, J7 3-641215-2, J8 3-641215-2, J9 3-641215-2, Q1 SSM6P49NU,LFPZ, Q10 FDG6303N, Q11 FDG6303N, Q12 FDG6303N, Q13 FDG6303N, Q14 FDG6303N, Q2 SSM6P49NU,LFPZ, Q3 FDG6303N, Q4 FDG6303N, Q5 FDC6506P, Q6 FDC6506P, Q7 FDG6303N, Q8 FDC6506P, Q9 FDG6303N, T1 PIC-OUT, T10 PIC-RPX, T11 PIC-RPX, T12 PIC-RPX, T13 PIC-RPX, T14 PIC-RPX, T15 PIC-OUT, T16 PIC-RPX, T17 PIC-RPX, T18 PIC-RPX, T19 PIC-RPX, T2 PIC-OUT, T20 PIC-OUT, T21 PIC-OUT, T22 PIC-RPX, T23 PIC-RPX, T24 PIC-RPX, T25 PIC-OUT, T26 PIC-OUT, T27 PIC-OUT, T28 PIC-OUT, T29 PIC-OUT, T3 PIC-RPX, T30 PIC-OUT, T31 PIC-OUT, T32 PIC-OUT, T33 PIC-OUT, T34 PIC-RPX, T35 PIC-RPX, T36 PIC-OUT, T37 PIN-AN, T38 PIN-AN, T39 PIN-AN, T4 PIC-OUT, T40 PIC-RPX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

Commit message: routing
a tone of routing work on the PCB, close to 35% done. camera and camera power routed, RAM routed, eeprom routed, started routing LAN.
TODO: find new BT connector, figure out how the IR LED's will be placed on PCB (wire or second connector), route LAN and rest of power, layout and route latch and door components.
Parts:
- added H3, H4, H5, H6, H7, H8: MOUNT-HOLE3.2, holes:MOUNT-HOLE3.2
- added J13: (no value), con-amp:MTA07-156
Connections:
- net +3.3V: now also J13.2
- net BT-RTS: now also J13.7
- net BT-RX: now also J13.3
- net BT-TX: now also J13.4
- net CON-LED: now also J13.6
- net DGND: now also J13.1
- net WAKE-SW: now also J13.5
Other:
- note added: "DOOR"
- note added: "ETHERNET CONTROL"
- note added: "IR_LED"
- note added: "RAM"
- note added: "VPS"
- note added: "replace BT connector"
Changed lines of the file:
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@@
 <?xml version="1.0" encoding="utf-8"?>
 <!DOCTYPE eagle SYSTEM "eagle.dtd">
-<eagle version="8.6.0">
+<eagle version="8.6.3">
 <drawing>
 <settings>
@@
 <part name="REF2" library="technol" deviceset="REF" device=""/>
 <part name="R132" library="DISCRETE" deviceset="R-0603" device="" value="1M"/>
+<part name="H3" library="holes" library_urn="urn:adsk.eagle:library:237" deviceset="MOUNT-HOLE" device="3.2" package3d_urn="urn:adsk.eagle:package:14275/1"/>
+<part name="H4" library="holes" library_urn="urn:adsk.eagle:library:237" deviceset="MOUNT-HOLE" device="3.2" package3d_urn="urn:adsk.eagle:package:14275/1"/>
+<part name="H5" library="holes" library_urn="urn:adsk.eagle:library:237" deviceset="MOUNT-HOLE" device="3.2" package3d_urn="urn:adsk.eagle:package:14275/1"/>
+<part name="H6" library="holes" library_urn="urn:adsk.eagle:library:237" deviceset="MOUNT-HOLE" device="3.2" package3d_urn="urn:adsk.eagle:package:14275/1"/>
+<part name="H7" library="holes" library_urn="urn:adsk.eagle:library:237" deviceset="MOUNT-HOLE" device="3.2" package3d_urn="urn:adsk.eagle:package:14275/1"/>
+<part name="H8" library="holes" library_urn="urn:adsk.eagle:library:237" deviceset="MOUNT-HOLE" device="3.2" package3d_urn="urn:adsk.eagle:package:14275/1"/>
+<part name="J13" library="con-amp" library_urn="urn:adsk.eagle:library:127" deviceset="MTA07-156" device=""/>
 </parts>
 <sheets>
@@
 <wire x1="579.12" y1="464.82" x2="579.12" y2="617.22" width="0.1524" layer="94" style="longdash"/>
 <wire x1="579.12" y1="617.22" x2="350.52" y2="617.22" width="0.1524" layer="94" style="longdash"/>
-<wire x1="589.28" y1="548.64" x2="589.28" y2="467.36" width="0.1524" layer="94" style="longdash"/>
-<wire x1="589.28" y1="467.36" x2="642.62" y2="467.36" width="0.1524" layer="94" style="longdash"/>
+<wire x1="581.66" y1="548.64" x2="581.66" y2="467.36" width="0.1524" layer="94" style="longdash"/>
+<wire x1="581.66" y1="467.36" x2="642.62" y2="467.36" width="0.1524" layer="94" style="longdash"/>
 <wire x1="642.62" y1="467.36" x2="642.62" y2="548.64" width="0.1524" layer="94" style="longdash"/>
-<wire x1="642.62" y1="548.64" x2="589.28" y2="548.64" width="0.1524" layer="94" style="longdash"/>
+<wire x1="642.62" y1="548.64" x2="581.66" y2="548.64" width="0.1524" layer="94" style="longdash"/>
 <wire x1="-165.1" y1="165.1" x2="-165.1" y2="462.28" width="0.1524" layer="94" style="longdash"/>
 <wire x1="-165.1" y1="462.28" x2="-434.34" y2="462.28" width="0.1524" layer="94" style="longdash"/>
 <wire x1="-434.34" y1="462.28" x2="-434.34" y2="165.1" width="0.1524" layer="94" style="longdash"/>
 <wire x1="-434.34" y1="165.1" x2="-165.1" y2="165.1" width="0.1524" layer="94" style="longdash"/>
+<text x="589.28" y="553.72" size="6.4516" layer="94">replace BT connector</text>
+<text x="-312.42" y="480.06" size="6.4516" layer="94">IR_LED</text>
+<text x="-139.7" y="477.52" size="6.4516" layer="94">DOOR</text>
+<text x="119.38" y="477.52" size="6.4516" layer="94">VPS</text>
+<text x="353.06" y="467.36" size="6.4516" layer="94">RAM</text>
+<text x="353.06" y="167.64" size="6.4516" layer="94">ETHERNET CONTROL</text>
 </plain>
 <instances>
@@
 <instance part="Q3" gate="-B" x="-248.92" y="515.62"/>
 <instance part="Q14" gate="-B" x="-172.72" y="515.62"/>
+<instance part="H3" gate="G$1" x="655.32" y="480.06"/>
+<instance part="H4" gate="G$1" x="662.94" y="480.06"/>
+<instance part="H5" gate="G$1" x="670.56" y="480.06"/>
+<instance part="H6" gate="G$1" x="655.32" y="472.44"/>
+<instance part="H7" gate="G$1" x="662.94" y="472.44"/>
+<instance part="H8" gate="G$1" x="670.56" y="472.44"/>
+<instance part="J13" gate="G$1" x="586.74" y="518.16" rot="MR270"/>
 </instances>
 <busses>
@@
 <pinref part="U$123" gate="G$1" pin="DGND"/>
 <pinref part="J14" gate="G$1" pin="1"/>
+<wire x1="601.98" y1="518.16" x2="589.28" y2="518.16" width="0.1524" layer="91"/>
+<junction x="601.98" y="518.16"/>
+<pinref part="J13" gate="G$1" pin="1"/>
 </segment>
 <segment>
@@
 <wire x1="622.3" y1="515.62" x2="622.3" y2="525.78" width="0.1524" layer="91"/>
 <junction x="614.68" y="515.62"/>
+<pinref part="J13" gate="G$1" pin="2"/>
+<wire x1="601.98" y1="515.62" x2="589.28" y2="515.62" width="0.1524" layer="91"/>
+<junction x="601.98" y="515.62"/>
 </segment>
 <segment>
@@
 <pinref part="J14" gate="G$1" pin="5"/>
 <pinref part="T42" gate="G$1" pin="TP"/>
+<pinref part="J13" gate="G$1" pin="5"/>
+<wire x1="601.98" y1="508" x2="589.28" y2="508" width="0.1524" layer="91"/>
+<junction x="601.98" y="508"/>
 </segment>
 <segment>
@@
 <pinref part="J14" gate="G$1" pin="6"/>
 <pinref part="T43" gate="G$1" pin="TP"/>
+<pinref part="J13" gate="G$1" pin="6"/>
+<wire x1="601.98" y1="505.46" x2="589.28" y2="505.46" width="0.1524" layer="91"/>
+<junction x="601.98" y="505.46"/>
 </segment>
 <segment>
@@
 <pinref part="J14" gate="G$1" pin="7"/>
 <pinref part="T44" gate="G$1" pin="TP"/>
+<pinref part="J13" gate="G$1" pin="7"/>
+<wire x1="601.98" y1="502.92" x2="589.28" y2="502.92" width="0.1524" layer="91"/>
+<junction x="601.98" y="502.92"/>
 </segment>
 <segment>
@@
 <pinref part="J14" gate="G$1" pin="3"/>
 <pinref part="T40" gate="G$1" pin="TP"/>
+<pinref part="J13" gate="G$1" pin="3"/>
+<wire x1="601.98" y1="513.08" x2="589.28" y2="513.08" width="0.1524" layer="91"/>
+<junction x="601.98" y="513.08"/>
 </segment>
 <segment>
@@
 <pinref part="J14" gate="G$1" pin="4"/>
 <pinref part="T41" gate="G$1" pin="TP"/>
+<pinref part="J13" gate="G$1" pin="4"/>
+<wire x1="601.98" y1="510.54" x2="589.28" y2="510.54" width="0.1524" layer="91"/>
+<junction x="601.98" y="510.54"/>
 </segment>
 <segment>
@@
 which will not be processed correctly with this version.
 </note>
+<note version="8.2" severity="warning">
+Since Version 8.2, EAGLE supports online libraries. The ids
+of those online libraries will not be understood (or retained)
+with this version.
+</note>
+<note version="8.3" severity="warning">
+Since Version 8.3, EAGLE supports URNs for individual library
+assets (packages, symbols, and devices). The URNs of those assets
+will not be understood (or retained) with this version.
+</note>
+<note version="8.3" severity="warning">
+Since Version 8.3, EAGLE supports the association of 3D packages
+with devices in libraries, schematics, and board files. Those 3D
+packages will not be understood (or retained) with this version.
+</note>
 </compatibility>
