File: ACB/ACB/ACB-R1.0-43-CH09/OLD/ACB Jr.q.brd (EAGLE design)
At the start: 63.5 x 226.8 mm, 391 parts, among them IC1 PIC32MX470F512L-I/PF, IC10 MAX9938HEUK+T, IC11 24LC32A-I/MS, IC12 SN65HVD12D, IC13 REF3025, IC14 TPD2E001DZDR, IC15 TPD2E001DZDR, IC16 MCP6042-I/MS, IC2 R1LV1616, IC3 74LVC573APW-TSSOP20, IC4 74LVC573APW-TSSOP20, IC5 TLV73315PDBV, IC6 MIC841LYC, IC7 24LC32A-I/MS, IC8 LT3971EMSE, IC9 AT25SF321-SSHD, J1 FH12A-24S-0.5SH, J10 3-641215-2, J11 DNP-DM3AT, J12 USB_A_180, J14 pin1x8, J15 pin2x8, J17 DNP-open-hole, J2 FH12A-24S-0.5SH, J3 RJ8-8-180, J4 RJ8-8-180, J5 MOLEX430450613, J6 MOLEX430450613, J7 3-641215-2, J8 3-641215-2, J9 3-641215-2, Q1 SSM6P49NU,LFPZ, Q10 FDG6303N, Q11 FDG6303N, Q12 FDG6303N, Q13 FDG6303N, Q14 FDG6303N, Q2 SSM6P49NU,LFPZ, Q3 FDG6303N, Q4 FDG6303N, Q5 FDC6506P, Q6 FDC6506P, Q7 FDG6303N, Q8 FDC6506P, Q9 FDG6303N, T1 PIC-OUT, T10 PIC-RPX, T11 PIC-RPX, T12 PIC-RPX, T13 PIC-RPX, T14 PIC-RPX, T15 PIC-OUT, T16 PIC-RPX, T17 PIC-RPX, T18 PIC-RPX, T19 PIC-RPX, T2 PIC-OUT, T20 PIC-OUT, T21 PIC-OUT, T22 PIC-RPX, T23 PIC-RPX, T24 PIC-RPX, T25 PIC-OUT, T26 PIC-OUT, T27 PIC-OUT, T28 PIC-OUT, T29 PIC-OUT, T3 PIC-RPX, T30 PIC-OUT, T31 PIC-OUT, T32 PIC-OUT, T33 PIC-OUT, T34 PIC-RPX, T35 PIC-RPX, T36 PIC-OUT, T37 PIN-AN, T38 PIN-AN, T39 PIN-AN, T4 PIC-OUT, T40 PIC-RPX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

Commit message: huge update
Added finished schematic for ACB Lite 3.1, ready for fab after Jaroslavs review.
Parts:
- removed C82: 1u, DISCRETE:0603
- removed O10, O11, O5, T22, T23, T24, T46: PIC-RPX, TESTPAD:TEMP-PAD
- removed PCB2: DNP-PCB-VPS, ACB:PCB-VPS
- removed T25, T26, T29: PIC-OUT, TESTPAD:TEMP-PAD
- added J16, J18: 3-641215-2, Tyco-U:3-641215-2
- added R120, R121, R133: 100R, DISCRETE:0603@1
- J11: value DNP-DM3AT -> 3-641215-2; device CON-Hirose-AON:DM3AT -> Tyco-U:3-641215-2
- J15: value pin2x8 -> 3-641215-2; device CON-pinHeader-AON:MA08-2 -> Tyco-U:3-641215-2
- R127: value 1M -> 100R
- moved J11 225.7 mm to (3.73, 145.8), flipped to the top
- moved J15 199.2 mm to (3.66, 152.0), turned to 270 degrees
- moved J7 181.9 mm to (11.1, 212.4), turned to 0 degrees
- moved J8 167.1 mm to (52.1, 213.5), turned to 180 degrees
- moved R67 163.6 mm to (3.90, 180.8), turned to 180 degrees
- moved C84 162.7 mm to (10.6, 184.0), turned to 270 degrees
- moved D7 161.0 mm to (18.7, 186.8), turned to 0 degrees
- moved PCB3 160.1 mm to (21.4, 191.6), turned to 180 degrees
- moved Q11 160.1 mm to (5.00, 178.5), turned to 90 degrees
- moved R64 157.3 mm to (5.00, 176.2), turned to 180 degrees
- moved C22 156.9 mm to (19.8, 184.1), turned to 180 degrees
- moved R54 155.6 mm to (5.00, 174.7), turned to 180 degrees
- moved R22 155.3 mm to (16.6, 181.3), turned to 270 degrees
- moved L9 154.8 mm to (26.1, 185.2), turned to 180 degrees
- moved C23 153.9 mm to (19.8, 181.8), turned to 180 degrees
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Connections:
- removed net EN: IC1.18, J15.8, O10.P$1, T25.P$1
- removed net IRQ: IC1.19, J15.3, O11.P$1, T24.P$1
- removed net NC-A15-2: IC1.42
- removed net SD-CS: IC1.9, J11.2, O5.P$1, R127.2, T29.P$1
- new net LATCH_SW_1: IC1.9, J11.1, R120.2
- new net LATCH_SW_2: IC1.18, J15.1, R127.2
- new net LATCH_SW_3: IC1.19, J16.1, R121.2
- new net LATCH_SW_4: IC1.42, J18.1, R133.2
- net +3.3V: now also R120.1, R121.1, R127.1, R133.1
- net +3.3V/VPS: no longer C82.1, J11.4, J15.1
- net /NCS: no longer J15.13, T26.P$1
- net /PRESENT: no longer J11.G2, T46.P$1
- net DGND: now also J11.2, J15.2, J16.2, J18.2; no longer C82.2, J11.6, J11.G1, J11.G3, J11.G4, J11.G5, J11.G6, J15.9, PCB2.VPS_PCB_1, R127.1
- net SCLK2-SPI: no longer J11.5, J15.12
- net SDI2-MISO: no longer J11.7, J15.11, T22.P$1
- net SDO2-MOSI: no longer J11.3, J15.14, T23.P$1
Routing:
- net INFRA1PWM: track 10.4 -> 147.6 mm, vias 1 -> 6
- net /3.3V2PWRON: track 5.99 -> 135.3 mm, vias 1 -> 4
- net /CAM-PWRON: track 5.70 -> 134.4 mm, vias 1 -> 6
- net BT-RTS: track 6.85 -> 131.9 mm, vias 0 -> 2
- net BT-TX: track 6.50 -> 131.4 mm, vias 1 -> 2
- net CON-LED: track 4.58 -> 122.3 mm, vias 1 -> 4
- net WAKE-SW: track 7.15 -> 117.1 mm, vias 1 -> 2
- net DOOR2IN: track 5.41 -> 114.4 mm, vias 1 -> 4
- net BT-RX: track 6.78 -> 113.6 mm, vias 1 -> 2
- net +3.3V: track 118.0 -> 212.1 mm, vias 8 -> 10
- net LATCH_SW_4: track 0.00 -> 89.3 mm, vias 0 -> 4
- net LATCH_SW_1: track 0.00 -> 83.4 mm
- net /MCLR: track 0.00 -> 77.3 mm, vias 0 -> 4
- net PGC: track 4.69 -> 76.7 mm, vias 0 -> 2
- net PGD: track 9.98 -> 79.0 mm, vias 0 -> 2
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- added copper zone on layer 1, net DGND-F
