File: ACB/ACB-LITE-3.2/ACB-Lite-1.0-J08.brd (EAGLE design)
At the start: 68.6 x 241.3 mm, 245 parts, among them IC1 PIC32MX470F512L-I/PF, IC10 MAX9938HEUK+T, IC11 24LC32A-I/MS, IC12 SN65HVD12D, IC13 REF3025, IC14 TPD2E001DZDR, IC15 TPD2E001DZDR, IC16 MCP6042-I/MS, IC2 L6227Q, IC3 LT3971EMSE, IC6 MIC841LYC, IC7 24LC32A-I/MS, IC9 AT25SF321-SSHD, J1 3-641215-2, J10 166087-4, J12 USB_B_180, J13 3-641215-2, J14 DNP-open-hole, J15 DNP-open-hole, J17 DNP-open-hole, J2 3-641215-2, J3 RJ8-8-180, J4 RJ8-8-180, J5 3-641215-2, J6 3-641215-2, J7 3-641215-2, J8 3-641215-5, J9 3-641215-5, Q1 SSM6P49NU,LFPZ, Q2 SSM6P49NU,LFPZ, Q3 FDC6330L, Q4 FDG6303N, Q5 FDC6506P, Q6 FDG6303N, Q7 FDC6506P, T1 PIC-OUT, T13 PIC-RPX, T14 PIC-RPX, T15 PIC-OUT, T27 PIC-OUT, T3 PIC-RPX, T32 PIC-OUT, T33 PIC-OUT, T36 PIC-OUT, T37 PIN-AN, T38 PIN-AN, T39 PIN-AN, T40 PIC-RPX, T41 PIC-RPX, T42 PIC-OUT, T43 PIC-RPX, T44 PIC-OUT, T45 PIC-RPX, T5 PIC-OUT, T7 PIC-OUT, X1 8MHz-5x3.2mm

Commit message: gen6 board
Parts:
- removed PCB1: PCB-ACB20, ACB:PCB-ACB20
Connections:
- net DGND: no longer PCB1.PAD_GND_1, PCB1.PAD_GND_2, PCB1.PAD_GND_3, PCB1.PAD_GND_4
Routing:
- net DGND: vias 266 -> 270
Changed lines of the file:
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@@
 <setting verticaltext="up"/>
 </settings>
-<grid distance="0.1" unitdist="mm" unit="mm" style="lines" multiple="10" display="yes" altdistance="0.05" altunitdist="mm" altunit="mm"/>
+<grid distance="0.05" unitdist="inch" unit="inch" style="lines" multiple="1" display="yes" altdistance="0.05" altunitdist="mm" altunit="mm"/>
 <layers>
 <layer number="1" name="Top" color="4" fill="1" visible="yes" active="yes"/>
@@
 <layer number="17" name="Pads" color="2" fill="1" visible="yes" active="yes"/>
 <layer number="18" name="Vias" color="2" fill="1" visible="yes" active="yes"/>
-<layer number="19" name="Unrouted" color="6" fill="10" visible="yes" active="yes"/>
+<layer number="19" name="Unrouted" color="6" fill="10" visible="no" active="yes"/>
 <layer number="20" name="Dimension" color="15" fill="1" visible="yes" active="yes"/>
 <layer number="21" name="tPlace" color="7" fill="1" visible="yes" active="yes"/>
-<layer number="22" name="bPlace" color="7" fill="1" visible="no" active="yes"/>
+<layer number="22" name="bPlace" color="7" fill="1" visible="yes" active="yes"/>
 <layer number="23" name="tOrigins" color="15" fill="1" visible="yes" active="yes"/>
 <layer number="24" name="bOrigins" color="15" fill="1" visible="no" active="yes"/>
-<layer number="25" name="tNames" color="7" fill="1" visible="no" active="yes"/>
+<layer number="25" name="tNames" color="7" fill="1" visible="yes" active="yes"/>
 <layer number="26" name="bNames" color="7" fill="1" visible="no" active="yes"/>
 <layer number="27" name="tValues" color="7" fill="1" visible="no" active="yes"/>
@@
 <layer number="29" name="tStop" color="7" fill="3" visible="no" active="yes"/>
 <layer number="30" name="bStop" color="7" fill="6" visible="no" active="yes"/>
-<layer number="31" name="tCream" color="6" fill="15" visible="yes" active="yes"/>
+<layer number="31" name="tCream" color="6" fill="15" visible="no" active="yes"/>
 <layer number="32" name="bCream" color="7" fill="5" visible="no" active="yes"/>
 <layer number="33" name="tFinish" color="6" fill="3" visible="no" active="yes"/>
@@
 <layer number="39" name="tKeepout" color="4" fill="11" visible="no" active="yes"/>
 <layer number="40" name="bKeepout" color="1" fill="11" visible="no" active="yes"/>
-<layer number="41" name="tRestrict" color="4" fill="10" visible="yes" active="yes"/>
-<layer number="42" name="bRestrict" color="1" fill="10" visible="yes" active="yes"/>
+<layer number="41" name="tRestrict" color="4" fill="10" visible="no" active="yes"/>
+<layer number="42" name="bRestrict" color="1" fill="10" visible="no" active="yes"/>
 <layer number="43" name="vRestrict" color="2" fill="10" visible="no" active="yes"/>
 <layer number="44" name="Drills" color="7" fill="1" visible="no" active="yes"/>
@@
 <layer number="106" name="bPlate" color="7" fill="1" visible="no" active="no"/>
 <layer number="107" name="Crop" color="7" fill="1" visible="no" active="no"/>
-<layer number="108" name="tOverlay" color="12" fill="1" visible="yes" active="yes"/>
+<layer number="108" name="tOverlay" color="12" fill="1" visible="no" active="yes"/>
 <layer number="110" name="110" color="7" fill="1" visible="no" active="no"/>
 <layer number="111" name="111" color="7" fill="1" visible="no" active="no"/>
@@
 <wire x1="21" y1="193" x2="20.8" y2="192.8" width="0.2" layer="41"/>
 <rectangle x1="11.9" y1="125.6" x2="13.1" y2="126.4" layer="108"/>
+<wire x1="-34.29" y1="0" x2="-13.97" y2="0" width="0" layer="20"/>
+<wire x1="-13.97" y1="0" x2="-13.97" y2="31.75" width="0" layer="20"/>
+<wire x1="-13.97" y1="31.75" x2="13.97" y2="31.75" width="0" layer="20"/>
+<wire x1="13.97" y1="31.75" x2="13.97" y2="0" width="0" layer="20"/>
+<wire x1="13.97" y1="0" x2="34.29" y2="0" width="0" layer="20"/>
+<wire x1="34.29" y1="0" x2="34.29" y2="241.3" width="0" layer="20"/>
+<wire x1="34.29" y1="241.3" x2="-34.29" y2="241.3" width="0" layer="20"/>
+<wire x1="-34.29" y1="241.3" x2="-34.29" y2="0" width="0" layer="20"/>
 </plain>
 <attributes>
@@
 <attribute name="NAME" x="22.4" y="224" size="1" layer="25" font="vector" ratio="12" align="bottom-center"/>
 </element>
-<element name="PCB1" library="ACB" package="PCB-ACB20" value="PCB-ACB20" x="0" y="0"/>
 <element name="J8" library="Tyco-U" package="3-641215-5" value="3-641215-5" x="14.5" y="237.7" rot="R180"/>
 <element name="J9" library="Tyco-U" package="3-641215-5" value="3-641215-5" x="-14.5" y="237.7" rot="R180"/>
@@
 <via x="29.9" y="81" extent="1-16" drill="0.3" diameter="0.8"/>
 <via x="33.2" y="77.6" extent="1-16" drill="0.3" diameter="0.8"/>
-<contactref element="PCB1" pad="PAD_GND_3"/>
-<contactref element="PCB1" pad="PAD_GND_4"/>
-<contactref element="PCB1" pad="PAD_GND_2"/>
-<contactref element="PCB1" pad="PAD_GND_1"/>
 <via x="-16.6" y="32.7" extent="1-16" drill="0.3" diameter="0.8"/>
 <via x="17.2" y="33.1" extent="1-16" drill="0.3" diameter="0.8"/>
@@
 <via x="11.1" y="87.65" extent="1-16" drill="0.3" diameter="0.8"/>
 <contactref element="R55" pad="2"/>
+<via x="-30.48" y="3.81" extent="1-16" drill="3.175" diameter="6.35"/>
+<via x="30.48" y="3.81" extent="1-16" drill="3.175" diameter="6.35"/>
+<via x="30.48" y="237.49" extent="1-16" drill="3.175" diameter="6.35"/>
+<via x="-30.48" y="237.49" extent="1-16" drill="3.175" diameter="6.35"/>
+<wire x1="-22.23" y1="237.7" x2="-30.48" y2="237.49" width="0" layer="19" extent="1-1"/>
 </signal>
 <signal name="SDO2-MOSI">
